File: kicad/ver2_top/ver1.kicad_pcb (KiCad board)
At the start: 2 copper layers, 233.6 x 106.5 mm, 46 parts, among them SW1 SW_PUSH, SW10 SW_PUSH, SW11 SW_PUSH, SW12 SW_PUSH, SW13 SW_PUSH, SW14 SW_PUSH, SW15 SW_PUSH, SW16 SW_PUSH, SW17 SW_PUSH, SW18 SW_PUSH, SW19 SW_PUSH, SW2 SW_PUSH, SW20 SW_PUSH, SW21 SW_PUSH, SW22 SW_PUSH, SW23 SW_PUSH, SW24 SW_PUSH, SW25 SW_PUSH, SW26 SW_PUSH, SW27 SW_PUSH, SW28 SW_PUSH, SW29 SW_PUSH, SW3 SW_PUSH, SW30 SW_PUSH, SW31 SW_PUSH, SW32 SW_PUSH, SW33 SW_PUSH, SW34 SW_PUSH, SW35 SW_PUSH, SW36 SW_PUSH, SW4 SW_PUSH, SW5 SW_PUSH, SW6 SW_PUSH, SW7 SW_PUSH, SW8 SW_PUSH, SW9 SW_PUSH

Commit message: add gbr file
Parts:
- moved Ref** 19.2 mm to (113.7, 73.0)
- moved Ref** 19.1 mm to (38.1, 59.7)
- moved Ref** 18.0 mm to (165.7, 72.4)
- moved Ref** 16.9 mm to (234.9, 60.3)
- moved Ref** 14.6 mm to (35.6, 78.7)
- moved Ref** 12.6 mm to (238.8, 79.4)
Changed lines of the file:
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@@
     (pad_to_mask_clearance 0)
     (pcbplotparams
-      (layerselection 0x00010fc_ffffffff)
+      (layerselection 0x00010f0_ffffffff)
       (plot_on_all_layers_selection 0x0000000_00000000)
       (disableapertmacros false)
@@
       (outputformat 1)
       (mirror false)
-      (drillshape 1)
+      (drillshape 0)
       (scaleselection 1)
       (outputdirectory "")
@@
   )
   (footprint "kbd_Hole:m2_Screw_Hole" (layer "F.Cu")
-    (at 170.5 55)
+    (at 165.735 72.39)
     (descr "Mounting Hole 2.2mm, no annular, M2")
     (tags "mounting hole 2.2mm no annular m2")
@@
   )
   (footprint "kbd_Hole:m2_Screw_Hole" (layer "F.Cu")
-    (at 226.8 45.5)
+    (at 234.95 60.325)
     (descr "Mounting Hole 2.2mm, no annular, M2")
     (tags "mounting hole 2.2mm no annular m2")
@@
   )
   (footprint "kbd_Hole:m2_Screw_Hole" (layer "F.Cu")
-    (at 42.3 91.7)
+    (at 35.56 78.74)
     (descr "Mounting Hole 2.2mm, no annular, M2")
     (tags "mounting hole 2.2mm no annular m2")
@@
   )
   (footprint "kbd_Hole:m2_Screw_Hole" (layer "F.Cu")
-    (at 106.8 55.1)
+    (at 113.665 73.025)
     (descr "Mounting Hole 2.2mm, no annular, M2")
     (tags "mounting hole 2.2mm no annular m2")
@@
   )
   (footprint "kbd_Hole:m2_Screw_Hole" (layer "F.Cu")
-    (at 50.5 45.1)
+    (at 38.1 59.69)
     (descr "Mounting Hole 2.2mm, no annular, M2")
     (tags "mounting hole 2.2mm no annular m2")
@@
   )
   (footprint "kbd_Hole:m2_Screw_Hole" (layer "F.Cu")
-    (at 235 91.4)
+    (at 238.76 79.375)
     (descr "Mounting Hole 2.2mm, no annular, M2")
     (tags "mounting hole 2.2mm no annular m2")
